File: FemtoSat/KiCadProjectFiles/KRUPS-FemtoSat.kicad_sch (KiCad schematic)
At the start: 55 parts, among them J1 B2P-VH-FB-B, J2 B2PS-VH, J3 USB_C_Receptacle_USB2.0_16P, J4 Conn_02x02, Q1 IRF7410, SW1 Enclosure Detector, U1 BME280, U2 ESP32-S3-WROOM-1-N16R8, U3 TSR_2-2450, U4 TPS61023, U5 E22-900M33S, U6 TPS2117, U7 LR62XE, U8 BNO086, U9 AZ1117-3.3

Commit message: Changed to Raspi Pico, 1W radio
- Swapped the ESP32 S3 WROOM to a Raspberry Pi Pico 2 W on both the FemtoSat and RocketStation
- Swapped to 1W LoRa module in place of the 2W EBYTE one
- bunch of layout, documentation, miscellaneous changes
Parts:
- removed C1: 22u, Capacitor_SMD:C_0805_2012Metric_Pad1.18x1.45mm_HandSolder, symbol Device:C
- removed C4: 0.1u, Capacitor_SMD:C_0603_1608Metric_Pad1.08x0.95mm_HandSolder, symbol Device:C
- removed C6: 100u, Capacitor_SMD:C_1206_3216Metric_Pad1.33x1.80mm_HandSolder, symbol Device:C
- removed D2: LED, Diode_SMD:D_0603_1608Metric_Pad1.05x0.95mm_HandSolder, symbol Device:LED
- removed H1, H2: MountingHole, MountingHole:MountingHole_2.2mm_M2, symbol Mechanical:MountingHole
- removed H3: MountingHole, MountingHole:MountingHole_2.2mm_M2_DIN965_Pad, symbol Mechanical:MountingHole
- removed J3: USB_C_Receptacle_USB2.0_16P, Connector_USB:USB_C_Receptacle_GCT_USB4110, symbol Connector:USB_C_Receptacle_USB2.0_16P
- removed J4: Conn_02x02, Connector_PinHeader_2.54mm:PinHeader_2x02_P2.54mm_Vertical, symbol Connector_Generic:Conn_02x02_Counter_Clockwise
- removed JP1, JP2: Jumper_2_Small_Open, TestPoint:TestPoint_2Pads_Pitch2.54mm_Drill0.8mm, symbol Jumper:Jumper_2_Small_Open
- removed R2: 10k, Resistor_SMD:R_0603_1608Metric_Pad0.98x0.95mm_HandSolder, symbol Device:R
- removed R3, R4: 5.1k, Resistor_SMD:R_0603_1608Metric_Pad0.98x0.95mm_HandSolder, symbol Device:R
- removed R8: 68, Resistor_SMD:R_0603_1608Metric_Pad0.98x0.95mm_HandSolder, symbol Device:R
- removed TP3: TestPoint, TestPoint:TestPoint_Pad_D2.0mm, symbol Connector:TestPoint
- removed TP4: TestPoint, TestPoint:TestPoint_Pad_2.0x2.0mm, symbol Connector:TestPoint
- removed U2: ESP32-S3-WROOM-1-N16R8, RF_Module:ESP32-S3-WROOM-2, symbol RF_Module:ESP32-S3-WROOM-2
- removed U5: E22-900M33S, KRUPS-FemtoSat:E22-XXXM33S, symbol KRUPS-FemtoSat:E22-900M33S
- added TP2: +5V, TestPoint:TestPoint_Pad_2.0x2.0mm, symbol Connector:TestPoint
- added U2: Pico_2_W, KRUPS-FemtoSat:RaspberryPi_Pico2_W_SMD, symbol KRUPS-FemtoSat:Pico_2_W
- TP1: value TestPoint -> GND; footprint TestPoint:TestPoint_Pad_D2.0mm -> TestPoint:TestPoint_Pad_2.0x2.0mm
- TP3: renamed from TP2; footprint TestPoint:TestPoint_Pad_1.0x1.0mm -> TestPoint:TestPoint_Pad_2.0x2.0mm
- U3: footprint Converter_DCDC:Converter_DCDC_TRACO_TSR-1_THT -> KRUPS-FemtoSat:CONV_TSR_2-2450
- U5: renamed from U7; now fitted
- renumbered C2 to C1, C13 to C10, C14 to C11, C3 to C2, C5 to C3, C7 to C4, C8 to C5, C9 to C6, C10 to C7, C11 to C8, C12 to C9, R5 to R2, R6 to R3, R7 to R4, R9 to R5, R10 to R6, R11 to R7, U8 to U7, U9 to U8
Connections:
- net IO43 is gone; now on net GND: TP1.1
- net +5V: now also TP2.1, U2.39 (VSYS)
- net BNO086_HINTN: now also U2.9 (GPIO6)
- net GND: now also U2.13 (GND), U2.18 (GND), U2.23 (GND), U2.28 (GND), U2.3 (GND), U2.33 (AGND), U2.38 (GND), U2.8 (GND)
- net I2C_SCL: now also U2.12 (GPIO9)
- net I2C_SDA: now also U2.11 (GPIO8)
- net LORA_BUSY: now also U2.29 (GPIO22)
- net LORA_DIO1: now also U2.31 (GPIO26_ADC0)
- net SPI_CLK: now also U2.24 (GPIO18)
- net SPI_MISO: now also U2.21 (GPIO16)
- net SPI_MOSI: now also U2.25 (GPIO19)
- net SPI_NSS: now also U2.22 (GPIO17)
- net ~{BNO086_RESET}: now also U2.10 (GPIO7)
- net ~{LORA_RESET}: now also U2.27 (GPIO21)
- net LORA_TXEN renamed LORA_ANTSW
- net LORA_ANTSW: now also U2.26 (GPIO20)
- no-connect marks 22 -> 24
Other:
- note added: "1W LoRa Module 868/915MHz"
- note added: "Raspberry Pi Pico 2 W RP2350A, 4MB Flash"
- note removed: "2W LoRa Module 868/915MHz"
- note removed: "3.3V power for an LR62XE"
- note removed: "Alternate 1W LoRa Module 915MHz"
- note removed: "ESP32 Restart will restart the chip when the jumper is shorted"
- note removed: "ESP32-S3-WROOM-1 16MB Flash, 8MB PSRAM SoM"
- note removed: "LORA_TXEN goes to the RF Switch it switches between TX and RX modes Datasheet doesnt say if it needs to be high or low to enable TX, so idk"
- note removed: "Only to be included if we can't use the Ebyte module Will be mounted via adapter board"
- note removed: "Technically, USB-C can provide more than enough current to power the entire board, but because there are situations where the USB port might not provide enough current (e.g. a weird USB A to C converter cable), and considering the fact that this is a one off design with an already existing wide voltage power input, I don't see any good reason to spend time dealing with extra USB power management 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"
- note removed: "USB Enable will allow the chip to be programmed over USB when shorted at startup Otherwise, the chip will default to the program stored in flash memory"
- note removed: "USB-C Connector NO POWER For programming/debugging"
- note removed: "WROOM-2 modules are currently out of stock so a WROOM-1 has been substituted. The only difference between the two is that the WROOM 2 has octal SPI flash/PSRAM. The WROOM-2 is otherwise pin compatible with this PCB."
- moved on the sheet: FID1, FID2, FID3, TP3
